Commit message: Update leo_with_visible_arm.urdf.xacro

File: Simulations/leo_with_visible_arm.urdf.xacro (robot description, xacro)
@@ -163,10 +163,9 @@
     <origin xyz="0.15 0 0.1" rpy="0 0 0"/>
   </joint>
-  <!-- Depth Camera Sensor Plugin -->
+  <!-- Depth Camera Sensor -->
   <gazebo reference="depth_camera_link">
-    <sensor name="depth_camera" type="depth_camera">
-      <update_rate>30</update_rate>
-      <gz_frame_id>depth_camera_link</gz_frame_id>
-      <camera>
+    <material>Gazebo/Black</material>
+    <sensor name="depth_camera" type="rgbd_camera">
+      <camera name="depth_camera">
         <horizontal_fov>1.047</horizontal_fov>
         <image>
@@ -179,8 +178,18 @@
           <far>10.0</far>
         </clip>
+        <noise>
+          <type>gaussian</type>
+          <mean>0.0</mean>
+          <stddev>0.007</stddev>
+        </noise>
+        <depth_camera>
+          <output>depths</output>
+        </depth_camera>
       </camera>
       <always_on>1</always_on>
+      <update_rate>30</update_rate>
       <visualize>true</visualize>
       <topic>depth_camera</topic>
+      <gz_frame_id>depth_camera_link</gz_frame_id>
     </sensor>
   </gazebo>
